File: ampli.kicad_pcb (KiCad board)
At the start: 2 copper layers, 52 parts, among them J2 Conn_01x02, J3 Conn_01x03, K1 Relay_1CT, Q1 2N907, Q10 Q_PNP_BCE, Q11 BD138, Q12 Q_NPN_BCE, Q13 2N2222, Q2 2N907, Q3 2N907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

Commit message: 1er placement des composants
Parts:
- moved Q3 220.5 mm to (80.0, 74.9), turned to 270 degrees
- moved Q7 212.5 mm to (86.4, 76.2)
- moved C4 203.6 mm to (87.6, 49.5), turned to 90 degrees
- moved Q2 196.3 mm to (95.2, 76.2)
- moved C7 194.4 mm to (95.2, 52.1)
- moved C5 191.5 mm to (74.9, 49.5), turned to 90 degrees
- moved Dz1 189.4 mm to (74.9, 58.4), turned to 270 degrees
- moved C1 187.6 mm to (90.2, 116.8)
- moved RV2 185.9 mm to (76.2, 102.9), turned to 90 degrees
- moved C6 185.5 mm to (95.2, 44.5)
- moved Q10 183.0 mm to (118.1, 45.7)
- moved Q1 182.4 mm to (85.1, 97.8), turned to 270 degrees
- moved Q6 180.4 mm to (95.2, 59.7)
- moved Q5 180.3 mm to (110.5, 85.1), turned to 270 degrees
- moved R1 179.8 mm to (85.1, 111.8), turned to 270 degrees
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
Commit message: pcb front
Parts:
- added D3: D, CmpAmpliAudio:D_DO-35_SOD27_P10.16mm_Horizontal, F.Cu at (74.9, 58.4)
- added D4: D, CmpAmpliAudio:D_DO-35_SOD27_P10.16mm_Horizontal, F.Cu at (78.7, 49.5)
- moved HS2 65.7 mm to (127.0, 45.7)
- moved R3 60.2 mm to (156.2, 108.0)
- moved R2 57.4 mm to (149.9, 108.0), turned to 270 degrees
- moved C10 54.6 mm to (170.2, 63.5)
- moved Dz1 49.6 mm to (77.5, 108.0), turned to 90 degrees
- moved R4 49.5 mm to (81.3, 108.0), turned to 0 degrees
- moved Q12 49.3 mm to (130.8, 48.3), turned to 90 degrees
- moved R15 49.3 mm to (158.8, 121.9), turned to 0 degrees
- moved C3 46.2 mm to (153.7, 31.8), turned to 270 degrees
- moved Q1 42.6 mm to (123.2, 116.8), turned to 0 degrees
- moved Q2 41.3 mm to (120.0, 109.2)
- moved R12 40.4 mm to (137.2, 62.2)
- moved R6 40.3 mm to (154.9, 100.3), turned to 0 degrees
- moved Q5 39.3 mm to (146.7, 100.3)
- moved Q3 35.5 mm to (102.8, 102.2)
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Routing:
- net -12V: track 0.00 -> 411.5 mm
- net (no net): track 411.5 -> 0.00 mm
