File: ampli.sch (KiCad schematic (older format))
At the start: 52 parts, among them J2 Conn_01x02, J3 Conn_01x03, K1 Relay_1CT, Q1 2N907, Q10 Q_PNP_BCE, Q11 BD138, Q12 Q_NPN_BCE, Q13 2N2222, Q2 2N907, Q3 2N907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

Commit message: schema
Parts:
- added D3, D4: D, CmpAmpliAudio:D_DO-35_SOD27_P10.16mm_Horizontal, symbol Device:D
Connections:
- net +12V: now also D3.1 (K)
- net -12V: now also D4.2 (A)
- net GND: now also D3.2 (A), D4.1 (K)
Changed lines of the file:
@@
 $EndComp
 Wire Wire Line
-	2950 6750 2350 6750
+	2950 6750 2700 6750
 Wire Wire Line
 	1450 6050 1850 6050
@@
 	0    1    1    0
 $EndComp
+$Comp
+L Device:D D3
+U 1 1 6075B0A6
+P 2700 6350
+F 0 "D3" V 2654 6430 50  0000 L CNN
+F 1 "D" V 2745 6430 50  0000 L CNN
+F 2 "CmpAmpliAudio:D_DO-35_SOD27_P10.16mm_Horizontal" H 2700 6350 50  0001 C CNN
+F 3 "~" H 2700 6350 50  0001 C CNN
+	1    2700 6350
+	0    1    1    0
+$EndComp
+$Comp
+L Device:D D4
+U 1 1 60762ECE
+P 2700 7000
+F 0 "D4" V 2654 7080 50  0000 L CNN
+F 1 "D" V 2745 7080 50  0000 L CNN
+F 2 "CmpAmpliAudio:D_DO-35_SOD27_P10.16mm_Horizontal" H 2700 7000 50  0001 C CNN
+F 3 "~" H 2700 7000 50  0001 C CNN
+	1    2700 7000
+	0    1    1    0
+$EndComp
+Wire Wire Line
+	2700 6500 2700 6750
+Connection ~ 2700 6750
+Wire Wire Line
+	2700 6750 2350 6750
+Wire Wire Line
+	2350 7300 2700 7300
+Wire Wire Line
+	2700 7300 2700 7150
+Connection ~ 2350 7300
+Wire Wire Line
+	2700 6850 2700 6750
+Wire Wire Line
+	2700 6200 2700 6050
+Wire Wire Line
+	2700 6050 2350 6050
+Connection ~ 2350 6050
 $EndSCHEMATC
